File: cad/pcb-v3/pcb-v5-routed-wip.kicad_pcb (KiCad board)
At the start: 4 copper layers, 20 x 19 mm, 50 parts

Commit message: pin U5 and get both: tight PCM cluster AND the good routing position
The two objectives were never actually in conflict -- I had been letting the
placer choose U5 and then arguing about the consequences.

U5's trial ranking optimises ONE thing (S1 -> BT1-2). Trial 8 wins that and
also allows a tight cluster, but the BOARD routes worse from there: gnd_taps
loses 7 pads instead of 4 and the filled result was 8 open with the F.Cu pour
back to 12 islands. Trial 27 routes well but, before the slot-candidate fix,
left C14 19.77 mm away.

With slot centres now available as candidates, pinning U5 to the trial-27
position gives BOTH:

    U5   (-3.70, -7.83)      the position that routed to 2 open pads
    C14   2.18 mm            was 19.77 -- the bypass now bypasses
    R9    2.25 mm
    R8    3.10 mm

Added TOUCHID_PIN_U5="x,y,rot" to pin U5 for exactly this kind of experiment.
The trial that wins on U5's own objective is not always the one the whole board
routes best, and the only way to find out is to build both -- ranking cannot
tell you, because the thing being ranked is not the thing that matters.

clearance 0 after push_off_pads (29 segments, 0 failures). Board is UNFILLED.
Parts:
- moved C13 8.20 mm to (-8.60, -2.65)
- moved C6 7.20 mm to (-8.60, -7.90)
- moved R8 5.55 mm to (-6.80, -7.90), turned to 0 degrees
- moved C12 4.40 mm to (-7.70, 7.85)
- moved R5 4.40 mm to (-7.05, 3.50)
- moved U5 3.55 mm to (-3.70, -7.90), turned to 0 degrees
- moved R9 2.65 mm to (-1.45, -7.90), turned to 90 degrees
- moved C10 1.76 mm to (6.00, 5.84)
- moved C3 1.76 mm to (6.00, 7.60)
- moved TP3 1.75 mm to (-0.97, -4.47)
- moved C14 0.90 mm to (-5.85, -8.20)
- moved C4 0.05 mm to (2.15, -7.90)
- moved C5 0.05 mm to (-0.55, -7.90)
- moved C9 0.05 mm to (0.35, -7.90)
- moved R6 0.05 mm to (1.25, -7.90)
Routing:
- net BL_FLAG: track 12.2 -> 27.5 mm, vias 3 -> 2
- net VBAT: track 25.8 -> 14.4 mm
- net PCM_VDD: track 10.6 -> 1.98 mm
- net VBAT_SENSE: track 16.2 -> 22.7 mm, vias 4 -> 2
- net VIN_DC: track 32.6 -> 26.4 mm, vias 6 -> 4
- net SENSOR_3V3: track 27.3 -> 32.5 mm, vias 2 -> 3
- net CELL_NEG: track 10.2 -> 5.31 mm
- net PCM_VM: track 5.31 -> 1.26 mm, vias 2 -> 0
- net VREF_SAMP: track 9.54 -> 5.95 mm, vias 3 -> 0
- net GND: track 8.12 -> 4.99 mm, vias 26 -> 29
- net VSTOR: track 44.9 -> 47.4 mm, vias 5 -> 6
- net VBAT_OK: track 23.2 -> 25.3 mm, vias 4 -> 5
- net HARV_2: track 14.7 -> 13.2 mm
- net SENSOR_WAKEUP: track 13.5 -> 14.8 mm
- net SENSOR_RX: track 17.2 -> 16.1 mm
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
Commit message: 4 -> 2 open, and check_drc is CLEAN for the first time
Pinned-U5 board, filled: 4 open. Closed by the tools that exist for it:
  island_via   ROV1.2  -- a via inside the pour island the pad actually sits in
  close_open   U2.18   -- 15.95 mm to VBAT's connected copper
Leaves ROK3.1 (VRDIV) and C7.2 (GND).

check_board 0 clearance violations, and check_drc reports NO VIOLATIONS AT ALL
-- the first fully clean DRC on this board. Previous runs always carried
phantoms from its net-number mis-resolution; there is nothing left for it to
mis-resolve.

The last two share one pocket, walled by the OK_HYST and VBAT_OV_SET tracks and
by each other's pads, with zero via sites. Promoting VRDIV into stage 1b was
tried: it fails on its own there (9/10, VRDIV open), so earlier is not the
answer for this one -- the pocket is the problem, not the order.

Board is UNFILLED (island_via's via and U2.18's route both landed after the
last fill).
Routing:
- net VBAT: track 14.4 -> 34.3 mm, vias 2 -> 5
- net GND: vias 29 -> 30
